Commit message: first commit

File: src/robot_description/urdf/erobot3.urdf (robot description, URDF)
Before this commit: robot eRobot3, 7 links, 6 joints
Links:
- link Link1: geometry collision mesh filename=package://robot_description/meshes/simplified_Link1.STL; visual mesh filename=package://robot_description/meshes/Link1.STL
- link Link2: geometry collision mesh filename=package://robot_description/meshes/simplified_Link2.STL; visual mesh filename=package://robot_description/meshes/Link2.STL
- link Link3: geometry collision mesh filename=package://robot_description/meshes/simplified_Link3.STL; visual mesh filename=package://robot_description/meshes/Link3.STL
- link Link4: geometry collision mesh filename=package://robot_description/meshes/simplified_Link4.STL; visual mesh filename=package://robot_description/meshes/Link4.STL
- link Link5: geometry collision mesh filename=package://robot_description/meshes/simplified_Link5.STL; visual mesh filename=package://robot_description/meshes/Link5.STL
- link Link6: geometry collision mesh filename=package://robot_description/meshes/simplified_Link6.STL; visual mesh filename=package://robot_description/meshes/Link6.STL
- link base_link: geometry collision mesh filename=package://robot_description/meshes/simplified_base_link.STL; visual mesh filename=package://robot_description/meshes/base_link.STL
